File: hardware/rx-pcb/bluetooth_test/rx-pcb.kicad_pcb (KiCad board)
At the start: 4 copper layers, 23.1 x 37.6 mm, 36 parts, among them J1 Conn_01x05_Pin, J2 Conn_01x04_Pin, J3 Conn_Coaxial_Small, J4 Conn_01x04_Pin, J5 Conn_01x02_Pin, SW1 SW_SPST, U1 STM32WB05KZV6TR, U2 STS4L-AD1B-R3, U3 LMT70AYFQR, X1 Q22FA12800025, X2 ABS07-32.768KHZ-1-T

Commit message: fixed merge errors, re updated rx-pcb
Parts:
- U2: footprint easyeda2kicad:DFN-4_L1.5-W1.5-P0.80-TL-EP -> rx-parts:DFN-4_L1.5-W1.5-P0.80-TL-EP
- U3: footprint easyeda2kicad:DSBGA-4_L0.8-W0.8-R2-C2-P0.40-BL -> rx-parts:DSBGA-4_L0.8-W0.8-R2-C2-P0.40-BL
- moved U3 5.12 mm to (164.2, 103.6)
Connections:
- net /RF/ANT renamed /ANT
- U1 pad 1: unconnected-(U1-PB3-Pad1) -> /TMP_A
- U1 pad 8: /TMP_A -> unconnected-(U1-PA0-Pad8)
