File: hardware/rx-pcb/power_harvester/power_harvester.kicad_sch (KiCad schematic)
At the start: 47 parts, among them J1 Conn_Coaxial_Small, J2 Conn_01x02_Pin, J3 Conn_Coaxial_Small, J4 Conn_Coaxial_Small

Commit message: fixed capacitance issue on harvester board
Parts:
- C1, C10, C2, C3, C9: footprint Capacitor_SMD:C_0603_1608Metric_Pad1.08x0.95mm_HandSolder -> Capacitor_SMD:C_0402_1005Metric
- C8: footprint Capacitor_SMD:C_0603_1608Metric_Pad1.08x0.95mm_HandSolder -> (none)
- D1, D2: value D -> JDH2S02SL
- D3, D4: value D_Zener -> SP4340L-01WTG
Other:
- moved on the sheet: D3, D4
Changed lines of the file:
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@@
 	)
 	(junction
-		(at 91.44 45.72)
-		(diameter 0)
-		(color 0 0 0 0)
-	)
-	(junction
 		(at 50.8 182.88)
 		(diameter 0)
@@
 	)
 	(junction
+		(at 83.82 45.72)
+		(diameter 0)
+		(color 0 0 0 0)
+	)
+	(junction
 		(at 92.71 113.03)
 		(diameter 0)
@@
 	(wire
 		(pts
-			(xy 91.44 64.77) (xy 91.44 66.04)
+			(xy 83.82 64.77) (xy 83.82 66.04)
 		)
 		(stroke
@@
 	(wire
 		(pts
-			(xy 91.44 45.72) (xy 91.44 48.26)
+			(xy 83.82 45.72) (xy 83.82 48.26)
 		)
 		(stroke
@@
 	(wire
 		(pts
-			(xy 68.58 45.72) (xy 91.44 45.72)
+			(xy 68.58 45.72) (xy 83.82 45.72)
 		)
 		(stroke
@@
 	(wire
 		(pts
-			(xy 91.44 55.88) (xy 91.44 57.15)
+			(xy 83.82 55.88) (xy 83.82 57.15)
 		)
 		(stroke
@@
 	(wire
 		(pts
-			(xy 91.44 45.72) (xy 109.22 45.72)
-		)
-		(stroke
-			(width 0)
-			(type default)
-		)
-	)
-	(wire
-		(pts
 			(xy 125.73 177.8) (xy 125.73 179.07)
 		)
@@
 	(wire
 		(pts
+			(xy 83.82 45.72) (xy 109.22 45.72)
+		)
+		(stroke
+			(width 0)
+			(type default)
+		)
+	)
+	(wire
+		(pts
 			(xy 54.61 45.72) (xy 54.61 48.26)
 		)
@@
 			)
 		)
-		(property "Value" "D"
+		(property "Value" "JDH2S02SL"
 			(at 147.32 54.6099 90)
 			(show_name no)
@@
 			)
 		)
-		(property "Footprint" "Capacitor_SMD:C_0603_1608Metric_Pad1.08x0.95mm_HandSolder"
+		(property "Footprint" "Capacitor_SMD:C_0402_1005Metric"
 			(at 139.7 44.7548 0)
 			(hide yes)
@@
 			)
 		)
-		(property "Footprint" "Capacitor_SMD:C_0603_1608Metric_Pad1.08x0.95mm_HandSolder"
+		(property "Footprint" "Capacitor_SMD:C_0402_1005Metric"
 			(at 69.5452 57.15 0)
 			(hide yes)
@@
 		(exclude_from_sim no)
 		(in_bom yes)
-		(on_board yes)
+		(on_board no)
 		(in_pos_files yes)
 		(dnp no)
@@
 			)
 		)
-		(property "Footprint" "Capacitor_SMD:C_0603_1608Metric_Pad1.08x0.95mm_HandSolder"
+		(property "Footprint" ""
 			(at 164.1348 49.53 0)
 			(hide yes)
@@
 			)
 		)
-		(property "Footprint" "Capacitor_SMD:C_0603_1608Metric_Pad1.08x0.95mm_HandSolder"
+		(property "Footprint" "Capacitor_SMD:C_0402_1005Metric"
 			(at 69.5452 67.31 0)
 			(hide yes)
@@
 	(symbol
 		(lib_id "power:GND")
-		(at 91.44 66.04 0)
+		(at 83.82 66.04 0)
 		(unit 1)
 		(body_style 1)
@@
 		(fields_autoplaced yes)
 		(property "Reference" "#PWR012"
-			(at 91.44 72.39 0)
+			(at 83.82 72.39 0)
 			(hide yes)
 			(show_name no)
@@
 		)
 		(property "Value" "GND"
-			(at 91.44 71.12 0)
+			(at 83.82 71.12 0)
 			(show_name no)
 			(do_not_autoplace no)
@@
 		)
 		(property "Footprint" ""
-			(at 91.44 66.04 0)
+			(at 83.82 66.04 0)
 			(hide yes)
 			(show_name no)
@@
 		)
 		(property "Datasheet" ""
-			(at 91.44 66.04 0)
+			(at 83.82 66.04 0)
 			(hide yes)
 			(show_name no)
@@
 		)
 		(property "Description" "Power symbol creates a global label with name \"GND\" , ground"
-			(at 91.44 66.04 0)
+			(at 83.82 66.04 0)
 			(hide yes)
 			(show_name no)
@@
 		(dnp no)
 		(property "Reference" "D2"
-			(at 153.67 51.054 0)
+			(at 153.67 40.132 0)
 			(show_name no)
 			(do_not_autoplace no)
@@
 			)
 		)
-		(property "Value" "D"
-			(at 153.67 53.594 0)
+		(property "Value" "JDH2S02SL"
+			(at 153.67 42.672 0)
 			(show_name no)
 			(do_not_autoplace no)
@@
 			)
 		)
-		(property "Footprint" "Capacitor_SMD:C_0603_1608Metric_Pad1.08x0.95mm_HandSolder"
+		(property "Footprint" "Capacitor_SMD:C_0402_1005Metric"
 			(at 49.2252 67.31 0)
 			(hide yes)
@@
 	(symbol
 		(lib_id "Device:D_Zener")
-		(at 91.44 60.96 270)
+		(at 83.82 60.96 270)
 		(unit 1)
 		(body_style 1)
@@
 		(fields_autoplaced yes)
 		(property "Reference" "D4"
-			(at 93.98 59.6899 90)
+			(at 86.36 59.6899 90)
 			(show_name no)
 			(do_not_autoplace no)
@@
 			)
 		)
-		(property "Value" "D_Zener"
-			(at 93.98 62.2299 90)
+		(property "Value" "SP4340L-01WTG"
+			(at 86.36 62.2299 90)
 			(show_name no)
 			(do_not_autoplace no)
@@
 		)
 		(property "Footprint" "Capacitor_SMD:C_0201_0603Metric"
-			(at 91.44 60.96 0)
+			(at 83.82 60.96 0)
 			(hide yes)
 			(show_name no)
@@
 		)
 		(property "Datasheet" ""
-			(at 91.44 60.96 0)
+			(at 83.82 60.96 0)
 			(hide yes)
 			(show_name no)
@@
 		)
 		(property "Description" "Zener diode"
-			(at 91.44 60.96 0)
+			(at 83.82 60.96 0)
 			(hide yes)
 			(show_name no)
@@
 			)
 		)
-		(property "Footprint" "Capacitor_SMD:C_0603_1608Metric_Pad1.08x0.95mm_HandSolder"
+		(property "Footprint" "Capacitor_SMD:C_0402_1005Metric"
 			(at 49.2252 57.15 0)
 			(hide yes)
@@
 	(symbol
 		(lib_id "Device:D_Zener")
-		(at 91.44 52.07 270)
+		(at 83.82 52.07 270)
 		(unit 1)
 		(body_style 1)
@@
 		(fields_autoplaced yes)
 		(property "Reference" "D3"
-			(at 93.98 50.7999 90)
+			(at 86.36 50.7999 90)
 			(show_name no)
 			(do_not_autoplace no)
@@
 			)
 		)
-		(property "Value" "D_Zener"
-			(at 93.98 53.3399 90)
+		(property "Value" "SP4340L-01WTG"
+			(at 86.36 53.3399 90)
 			(show_name no)
 			(do_not_autoplace no)
@@
 		)
 		(property "Footprint" "Capacitor_SMD:C_0201_0603Metric"
-			(at 91.44 52.07 0)
+			(at 83.82 52.07 0)
 			(hide yes)
 			(show_name no)
@@
 		)
 		(property "Datasheet" ""
-			(at 91.44 52.07 0)
+			(at 83.82 52.07 0)
 			(hide yes)
 			(show_name no)
@@
 		)
 		(property "Description" "Zener diode"
-			(at 91.44 52.07 0)
+			(at 83.82 52.07 0)
 			(hide yes)
 			(show_name no)
